Commit message: add colors

File: ezgripper_driver/urdf/ezgripper_dual_gen2_plus_articulated.urdf.xacro (robot description, xacro)
@@ -1,6 +1,11 @@
 <?xml version="1.0" encoding="UTF-8"?>
 <robot name="ezgripper" xmlns:xacro="http://ros.org/wiki/xacro">
-<!--xacro:macro name="ezgripper" params="*origin"-->
 <xacro:macro name="ezgripper_dual" params="prefix parent_link *origin">
+    <material name="${prefix}White_Plastic">
+      <color rgba="0.9 0.9 0.9 1.0"/>
+    </material>
+    <material name="${prefix}Black_Plastic">
+      <color rgba="0.1 0.1 0.1 1.0"/>
+    </material>
     <!-- links -->
     <link name="${prefix}_ezgripper_palm_link">
@@ -10,4 +15,5 @@
           <mesh filename="package://ezgripper_driver/meshes/ezgripper_gen2_plus/SAKE_Palm_Dual_Gen2_simple.stl"/>
         </geometry>
+        <material name="${prefix}Black_Plastic"/>
       </visual>
       <collision>
@@ -53,4 +59,5 @@
           <mesh filename="package://ezgripper_driver/meshes/ezgripper_gen2_plus/SAKE_Finger_L1_Gen2_simple.stl"/>
         </geometry>
+        <material name="${prefix}White_Plastic"/>
       </visual>
       <collision>
@@ -73,4 +80,5 @@
           <mesh filename="package://ezgripper_driver/meshes/ezgripper_gen2_plus/SAKE_Finger_L2_Gen2_simple.stl"/>
         </geometry>
+        <material name="${prefix}White_Plastic"/>
       </visual>
       <collision>
@@ -93,4 +101,5 @@
           <mesh filename="package://ezgripper_driver/meshes/ezgripper_gen2_plus/SAKE_Finger_L2_Pad_simple.stl"/>
         </geometry>
+        <material name="${prefix}White_Plastic"/>
       </visual>
       <collision>

File: ezgripper_driver/urdf/ezgripper_dual_gen2_plus_standalone.urdf.xacro (robot description, xacro)
@@ -1,4 +1,4 @@
 <?xml version="1.0" encoding="UTF-8"?>
-<robot name="ezgripper_stand_alone" xmlns:xacro="http://www.ros.org/wiki/xacro">
+<robot name="ezgripper_stand_alone" xmlns:xacro="http://ros.org/wiki/xacro">
 <xacro:property name="ezgripper_offset_x" value="0.0"/>
 <xacro:property name="ezgripper_offset_y" value="0.0"/>
@@ -7,5 +7,5 @@
 <!-- Add the gripper -->
 <ezgripper_dual prefix="left" parent_link="base_link">
-<origin xyz="${ezgripper_offset_x} ${ezgripper_offset_y} ${ezgripper_offset_z}" rpy="0 0 0"/>
+  <origin xyz="${ezgripper_offset_x} ${ezgripper_offset_y} ${ezgripper_offset_z}" rpy="0 0 0"/>
 </ezgripper_dual>
 <link name="world"/>

Commit message: ezgripper: use White Plastic

File: ezgripper_driver/urdf/ezgripper_dual_gen2_plus_articulated.urdf.xacro (robot description, xacro)
@@ -15,5 +15,5 @@
           <mesh filename="package://ezgripper_driver/meshes/ezgripper_gen2_plus/SAKE_Palm_Dual_Gen2_simple.stl"/>
         </geometry>
-        <material name="${prefix}Black_Plastic"/>
+        <material name="${prefix}White_Plastic"/>
       </visual>
       <collision>
