Commit message: update project for noetic

File: ezgripper_driver/urdf/ezgripper_dual_articulated.urdf.xacro (robot description, xacro)
@@ -29,15 +29,15 @@
         <limit effort="0" lower="-1.57075" upper="0.25" velocity="3.67"/>
     </joint>
-    <ezgripper_finger_L1 prefix="${prefix}" postfix="1" reflect="1" />
-    <ezgripper_finger_L1 prefix="${prefix}" postfix="2" reflect="1" />
-    <ezgripper_finger_L2 prefix="${prefix}" postfix="1" reflect="1" />
-    <ezgripper_finger_L2 prefix="${prefix}" postfix="2" reflect="1" />
-    <ezgripper_knuckle_palm_L1 prefix="${prefix}" postfix="1" reflectY="1" reflectZ="1" reflectR="1" mimic_test="false"/>
-    <ezgripper_knuckle_palm_L1 prefix="${prefix}" postfix="2" reflectY="-1" reflectZ="1" reflectR="-1" mimic_test="true"/>
-    <ezgripper_knuckle_L1_L2 prefix="${prefix}" postfix="1" reflectY="1" reflectZ="1" reflectR="1" mimic_test="false"/>
-    <ezgripper_knuckle_L1_L2 prefix="${prefix}" postfix="2" reflectY="-1" reflectZ="1" reflectR="-1" mimic_test="true"/>
-    <ezgripper_knuckle_trans prefix="${prefix}" postfix="1"/>
-    <ezgripper_knuckle_trans prefix="${prefix}" postfix="2"/>
-    <gazebo_knuckle_jsp prefix="${prefix}" />
+    <xacro:ezgripper_finger_L1 prefix="${prefix}" postfix="1" reflect="1" />
+    <xacro:ezgripper_finger_L1 prefix="${prefix}" postfix="2" reflect="1" />
+    <xacro:ezgripper_finger_L2 prefix="${prefix}" postfix="1" reflect="1" />
+    <xacro:ezgripper_finger_L2 prefix="${prefix}" postfix="2" reflect="1" />
+    <xacro:ezgripper_knuckle_palm_L1 prefix="${prefix}" postfix="1" reflectY="1" reflectZ="1" reflectR="1" mimic_test="false"/>
+    <xacro:ezgripper_knuckle_palm_L1 prefix="${prefix}" postfix="2" reflectY="-1" reflectZ="1" reflectR="-1" mimic_test="true"/>
+    <xacro:ezgripper_knuckle_L1_L2 prefix="${prefix}" postfix="1" reflectY="1" reflectZ="1" reflectR="1" mimic_test="false"/>
+    <xacro:ezgripper_knuckle_L1_L2 prefix="${prefix}" postfix="2" reflectY="-1" reflectZ="1" reflectR="-1" mimic_test="true"/>
+    <xacro:ezgripper_knuckle_trans prefix="${prefix}" postfix="1"/>
+    <xacro:ezgripper_knuckle_trans prefix="${prefix}" postfix="2"/>
+    <xacro:gazebo_knuckle_jsp prefix="${prefix}" />
 </xacro:macro>
 <xacro:macro name="ezgripper_finger_L1" params="prefix postfix reflect">

File: ezgripper_driver/urdf/ezgripper_dual_gen2.urdf.xacro (robot description, xacro)
@@ -29,11 +29,11 @@
         <limit effort="0" lower="-1.57075" upper="0.25" velocity="3.67"/>
     </joint>
-    <ezgripper_finger prefix="${prefix}" postfix="1" reflect="1" />
-    <ezgripper_finger prefix="${prefix}" postfix="2" reflect="1" />
-    <ezgripper_knuckle prefix="${prefix}" postfix="1" reflectY="1" reflectZ="1" reflectR="1" mimic_test="false"/>
-    <ezgripper_knuckle prefix="${prefix}" postfix="2" reflectY="-1" reflectZ="1" reflectR="-1" mimic_test="true"/>
-    <ezgripper_knuckle_trans prefix="${prefix}" postfix="1"/>
-    <ezgripper_knuckle_trans prefix="${prefix}" postfix="2"/>
-    <gazebo_knuckle_jsp prefix="${prefix}" />
+    <xacro:ezgripper_finger prefix="${prefix}" postfix="1" reflect="1" />
+    <xacro:ezgripper_finger prefix="${prefix}" postfix="2" reflect="1" />
+    <xacro:ezgripper_knuckle prefix="${prefix}" postfix="1" reflectY="1" reflectZ="1" reflectR="1" mimic_test="false"/>
+    <xacro:ezgripper_knuckle prefix="${prefix}" postfix="2" reflectY="-1" reflectZ="1" reflectR="-1" mimic_test="true"/>
+    <xacro:ezgripper_knuckle_trans prefix="${prefix}" postfix="1"/>
+    <xacro:ezgripper_knuckle_trans prefix="${prefix}" postfix="2"/>
+    <xacro:gazebo_knuckle_jsp prefix="${prefix}" />
 </xacro:macro>
 <xacro:macro name="ezgripper_finger" params="prefix postfix reflect">

File: ezgripper_driver/urdf/ezgripper_dual_gen2_articulated.urdf.xacro (robot description, xacro)
@@ -30,14 +30,14 @@
         <limit effort="0" lower="-1.57075" upper="0.25" velocity="3.67"/>
     </joint>
-    <ezgripper_finger_L1 prefix="${prefix}" postfix="1" reflect="1" />
-    <ezgripper_finger_L1 prefix="${prefix}" postfix="2" reflect="1" />
-    <ezgripper_finger_L2 prefix="${prefix}" postfix="1" reflect="1" />
-    <ezgripper_finger_L2 prefix="${prefix}" postfix="2" reflect="1" />
-    <ezgripper_knuckle_palm_L1 prefix="${prefix}" postfix="1" reflectY="1" reflectZ="1" reflectR="1" mimic_test="false"/>
-    <ezgripper_knuckle_palm_L1 prefix="${prefix}" postfix="2" reflectY="-1" reflectZ="1" reflectR="-1" mimic_test="true"/>
-    <ezgripper_knuckle_L1_L2 prefix="${prefix}" postfix="1" reflectY="1" reflectZ="1" reflectR="-1" mimic_test="false"/>
-    <ezgripper_knuckle_L1_L2 prefix="${prefix}" postfix="2" reflectY="-1" reflectZ="1" reflectR="1" mimic_test="true"/>
-    <ezgripper_knuckle_trans prefix="${prefix}" postfix="L1_L2_1"/>
-    <gazebo_knuckle_jsp prefix="${prefix}" />
+    <xacro:ezgripper_finger_L1 prefix="${prefix}" postfix="1" reflect="1" />
+    <xacro:ezgripper_finger_L1 prefix="${prefix}" postfix="2" reflect="1" />
+    <xacro:ezgripper_finger_L2 prefix="${prefix}" postfix="1" reflect="1" />
+    <xacro:ezgripper_finger_L2 prefix="${prefix}" postfix="2" reflect="1" />
+    <xacro:ezgripper_knuckle_palm_L1 prefix="${prefix}" postfix="1" reflectY="1" reflectZ="1" reflectR="1" mimic_test="false"/>
+    <xacro:ezgripper_knuckle_palm_L1 prefix="${prefix}" postfix="2" reflectY="-1" reflectZ="1" reflectR="-1" mimic_test="true"/>
+    <xacro:ezgripper_knuckle_L1_L2 prefix="${prefix}" postfix="1" reflectY="1" reflectZ="1" reflectR="-1" mimic_test="false"/>
+    <xacro:ezgripper_knuckle_L1_L2 prefix="${prefix}" postfix="2" reflectY="-1" reflectZ="1" reflectR="1" mimic_test="true"/>
+    <xacro:ezgripper_knuckle_trans prefix="${prefix}" postfix="L1_L2_1"/>
+    <xacro:gazebo_knuckle_jsp prefix="${prefix}" />
 </xacro:macro>
 <xacro:macro name="ezgripper_finger_L1" params="prefix postfix reflect">

File: ezgripper_driver/urdf/ezgripper_dual_gen2_plus_articulated.urdf.xacro (robot description, xacro)
@@ -36,19 +36,19 @@
         <limit effort="0" lower="-1.57075" upper="0.25" velocity="3.67"/>
     </joint>
-    <ezgripper_finger_L1 prefix="${prefix}" postfix="1" reflect="1" />
-    <ezgripper_finger_L1 prefix="${prefix}" postfix="2" reflect="1" />
-    <ezgripper_finger_L2 prefix="${prefix}" postfix="1" reflect="1" />
-    <ezgripper_finger_L2 prefix="${prefix}" postfix="2" reflect="1" />
-    <ezgripper_finger_L2_pad prefix="${prefix}" postfix="1" reflect="1" />
-    <ezgripper_finger_L2_pad prefix="${prefix}" postfix="2" reflect="1" />
-    <ezgripper_knuckle_palm_L1 prefix="${prefix}" postfix="1" reflectY="1" reflectZ="1" reflectR="1" mimic_test="false"/>
-    <ezgripper_knuckle_palm_L1 prefix="${prefix}" postfix="2" reflectY="-1" reflectZ="1" reflectR="-1" mimic_test="true"/>
-    <ezgripper_knuckle_L1_L2 prefix="${prefix}" postfix="1" reflectY="1" reflectZ="1" reflectR="-1" mimic_test="false"/>
-    <ezgripper_knuckle_L1_L2 prefix="${prefix}" postfix="2" reflectY="-1" reflectZ="1" reflectR="1" mimic_test="true"/>
-    <ezgripper_mount_L2 prefix="${prefix}" postfix="1" reflectY="1" reflectZ="1" reflectR="-1" mimic_test="false"/>
-    <ezgripper_mount_L2 prefix="${prefix}" postfix="2" reflectY="-1" reflectZ="1" reflectR="1" mimic_test="true"/>
-    <ezgripper_knuckle_trans prefix="${prefix}" postfix="L1_L2_1"/>
-    <ezgripper_knuckle_trans prefix="${prefix}" postfix="L1_L2_2"/>
-    <gazebo_knuckle_jsp prefix="${prefix}" />
+    <xacro:ezgripper_finger_L1 prefix="${prefix}" postfix="1" reflect="1" />
+    <xacro:ezgripper_finger_L1 prefix="${prefix}" postfix="2" reflect="1" />
+    <xacro:ezgripper_finger_L2 prefix="${prefix}" postfix="1" reflect="1" />
+    <xacro:ezgripper_finger_L2 prefix="${prefix}" postfix="2" reflect="1" />
+    <xacro:ezgripper_finger_L2_pad prefix="${prefix}" postfix="1" reflect="1" />
+    <xacro:ezgripper_finger_L2_pad prefix="${prefix}" postfix="2" reflect="1" />
+    <xacro:ezgripper_knuckle_palm_L1 prefix="${prefix}" postfix="1" reflectY="1" reflectZ="1" reflectR="1" mimic_test="false"/>
+    <xacro:ezgripper_knuckle_palm_L1 prefix="${prefix}" postfix="2" reflectY="-1" reflectZ="1" reflectR="-1" mimic_test="true"/>
+    <xacro:ezgripper_knuckle_L1_L2 prefix="${prefix}" postfix="1" reflectY="1" reflectZ="1" reflectR="-1" mimic_test="false"/>
+    <xacro:ezgripper_knuckle_L1_L2 prefix="${prefix}" postfix="2" reflectY="-1" reflectZ="1" reflectR="1" mimic_test="true"/>
+    <xacro:ezgripper_mount_L2 prefix="${prefix}" postfix="1" reflectY="1" reflectZ="1" reflectR="-1" mimic_test="false"/>
+    <xacro:ezgripper_mount_L2 prefix="${prefix}" postfix="2" reflectY="-1" reflectZ="1" reflectR="1" mimic_test="true"/>
+    <xacro:ezgripper_knuckle_trans prefix="${prefix}" postfix="L1_L2_1"/>
+    <xacro:ezgripper_knuckle_trans prefix="${prefix}" postfix="L1_L2_2"/>
+    <xacro:gazebo_knuckle_jsp prefix="${prefix}" />
 </xacro:macro>
 <xacro:macro name="ezgripper_finger_L1" params="prefix postfix reflect">

File: ezgripper_driver/urdf/ezgripper_dual_gen2_plus_cam_articulated.urdf.xacro (robot description, xacro)
@@ -33,19 +33,19 @@
         <limit effort="0" lower="-1.57075" upper="0.25" velocity="3.67"/>
     </joint>
-    <ezgripper_finger_L1 prefix="${prefix}" postfix="1" reflect="1" />
-    <ezgripper_finger_L1 prefix="${prefix}" postfix="2" reflect="1" />
-    <ezgripper_finger_L2 prefix="${prefix}" postfix="1" reflect="1" />
-    <ezgripper_finger_L2 prefix="${prefix}" postfix="2" reflect="1" />
-    <ezgripper_finger_L2_pad prefix="${prefix}" postfix="1" reflect="1" />
-    <ezgripper_finger_L2_pad prefix="${prefix}" postfix="2" reflect="1" />
-    <ezgripper_knuckle_palm_L1 prefix="${prefix}" postfix="1" reflectY="1" reflectZ="1" reflectR="1" mimic_test="false"/>
-    <ezgripper_knuckle_palm_L1 prefix="${prefix}" postfix="2" reflectY="-1" reflectZ="1" reflectR="-1" mimic_test="true"/>
-    <ezgripper_knuckle_L1_L2 prefix="${prefix}" postfix="1" reflectY="1" reflectZ="1" reflectR="-1" mimic_test="false"/>
-    <ezgripper_knuckle_L1_L2 prefix="${prefix}" postfix="2" reflectY="-1" reflectZ="1" reflectR="1" mimic_test="true"/>
-    <ezgripper_mount_L2 prefix="${prefix}" postfix="1" reflectY="1" reflectZ="1" reflectR="-1" mimic_test="false"/>
-    <ezgripper_mount_L2 prefix="${prefix}" postfix="2" reflectY="-1" reflectZ="1" reflectR="1" mimic_test="true"/>
-    <ezgripper_knuckle_trans prefix="${prefix}" postfix="L1_L2_1"/>
-    <ezgripper_knuckle_trans prefix="${prefix}" postfix="L1_L2_2"/>
-    <gazebo_knuckle_jsp prefix="${prefix}" />
+    <xacro:ezgripper_finger_L1 prefix="${prefix}" postfix="1" reflect="1" />
+    <xacro:ezgripper_finger_L1 prefix="${prefix}" postfix="2" reflect="1" />
+    <xacro:ezgripper_finger_L2 prefix="${prefix}" postfix="1" reflect="1" />
+    <xacro:ezgripper_finger_L2 prefix="${prefix}" postfix="2" reflect="1" />
+    <xacro:ezgripper_finger_L2_pad prefix="${prefix}" postfix="1" reflect="1" />
+    <xacro:ezgripper_finger_L2_pad prefix="${prefix}" postfix="2" reflect="1" />
+    <xacro:ezgripper_knuckle_palm_L1 prefix="${prefix}" postfix="1" reflectY="1" reflectZ="1" reflectR="1" mimic_test="false"/>
+    <xacro:ezgripper_knuckle_palm_L1 prefix="${prefix}" postfix="2" reflectY="-1" reflectZ="1" reflectR="-1" mimic_test="true"/>
+    <xacro:ezgripper_knuckle_L1_L2 prefix="${prefix}" postfix="1" reflectY="1" reflectZ="1" reflectR="-1" mimic_test="false"/>
+    <xacro:ezgripper_knuckle_L1_L2 prefix="${prefix}" postfix="2" reflectY="-1" reflectZ="1" reflectR="1" mimic_test="true"/>
+    <xacro:ezgripper_mount_L2 prefix="${prefix}" postfix="1" reflectY="1" reflectZ="1" reflectR="-1" mimic_test="false"/>
+    <xacro:ezgripper_mount_L2 prefix="${prefix}" postfix="2" reflectY="-1" reflectZ="1" reflectR="1" mimic_test="true"/>
+    <xacro:ezgripper_knuckle_trans prefix="${prefix}" postfix="L1_L2_1"/>
+    <xacro:ezgripper_knuckle_trans prefix="${prefix}" postfix="L1_L2_2"/>
+    <xacro:gazebo_knuckle_jsp prefix="${prefix}" />
 </xacro:macro>
 <xacro:macro name="ezgripper_finger_L1" params="prefix postfix reflect">

File: ezgripper_driver/urdf/ezgripper_dual_gen2_plus_standalone.urdf.xacro (robot description, xacro)
@@ -6,7 +6,10 @@
 <xacro:include filename="$(find ezgripper_driver)/urdf/ezgripper_dual_gen2_plus_articulated.urdf.xacro"/>
 <!-- Add the gripper -->
-<ezgripper_dual prefix="main" parent_link="base_link">
+<xacro:ezgripper_dual prefix="main" parent_link="base_link">
   <origin xyz="${ezgripper_offset_x} ${ezgripper_offset_y} ${ezgripper_offset_z}" rpy="0 0 0"/>
-</ezgripper_dual>
+</xacro:ezgripper_dual>
+<material name="red">
+  <color rgba="0.7 0.0 0.0 0.99"/>
+</material>
 <link name="world"/>
 <joint name="fixed" type="fixed">

File: ezgripper_driver/urdf/ezgripper_dual_gen2_standalone.urdf.xacro (robot description, xacro)
@@ -6,7 +6,10 @@
 <xacro:include filename="$(find ezgripper_driver)/urdf/ezgripper_dual_gen2_articulated.urdf.xacro"/>
 <!-- Add the gripper -->
-<ezgripper_dual prefix="left" parent_link="base_link">
+<xacro:ezgripper_dual prefix="left" parent_link="base_link">
 <origin xyz="${ezgripper_offset_x} ${ezgripper_offset_y} ${ezgripper_offset_z}" rpy="0 0 0"/>
-</ezgripper_dual>
+</xacro:ezgripper_dual>
+<material name="red">
+  <color rgba="0.7 0.0 0.0 0.99"/>
+</material>
 <link name="world"/>
 <joint name="fixed" type="fixed">

File: ezgripper_driver/urdf/ezgripper_dual_standalone.urdf.xacro (robot description, xacro)
@@ -6,7 +6,10 @@
 <xacro:include filename="$(find ezgripper_driver)/urdf/ezgripper_dual.urdf.xacro"/>
 <!-- Add the gripper -->
-<ezgripper_dual prefix="left" parent_link="base_link">
+<xacro:ezgripper_dual prefix="left" parent_link="base_link">
 <origin xyz="${ezgripper_offset_x} ${ezgripper_offset_y} ${ezgripper_offset_z}" rpy="0 0 0"/>
-</ezgripper_dual>
+</xacro:ezgripper_dual>
+<material name="red">
+  <color rgba="0.7 0.0 0.0 0.99"/>
+</material>
 <link name="world"/>
 <joint name="fixed" type="fixed">

File: ezgripper_driver/urdf/ezgripper_quad.urdf.xacro (robot description, xacro)
@@ -28,17 +28,17 @@
         <limit effort="0" lower="-1.57075" upper="0.25" velocity="3.67"/>
     </joint>
-    <ezgripper_finger prefix="${prefix}" postfix="1" reflect="1"/>
-    <ezgripper_finger prefix="${prefix}" postfix="2" reflect="1"/>
-    <ezgripper_finger prefix="${prefix}" postfix="3" reflect="1"/>
-    <ezgripper_finger prefix="${prefix}" postfix="4" reflect="1"/>
-    <ezgripper_knuckle prefix="${prefix}" postfix="1" reflectY="1" reflectZ="1" reflectR="1" mimic_test="false"/>
-    <ezgripper_knuckle prefix="${prefix}" postfix="2" reflectY="-1" reflectZ="1" reflectR="-1" mimic_test="true"/>
-    <ezgripper_knuckle prefix="${prefix}" postfix="3" reflectY="1" reflectZ="-1" reflectR="1" mimic_test="true"/>
-    <ezgripper_knuckle prefix="${prefix}" postfix="4" reflectY="-1" reflectZ="-1" reflectR="-1" mimic_test="true"/>
-    <ezgripper_knuckle_trans prefix="${prefix}" postfix="1"/>
-    <ezgripper_knuckle_trans prefix="${prefix}" postfix="2"/>
-    <ezgripper_knuckle_trans prefix="${prefix}" postfix="3"/>
-    <ezgripper_knuckle_trans prefix="${prefix}" postfix="4"/>
-    <gazebo_knuckle_jsp prefix="${prefix}" />
+    <xacro:ezgripper_finger prefix="${prefix}" postfix="1" reflect="1"/>
+    <xacro:ezgripper_finger prefix="${prefix}" postfix="2" reflect="1"/>
+    <xacro:ezgripper_finger prefix="${prefix}" postfix="3" reflect="1"/>
+    <xacro:ezgripper_finger prefix="${prefix}" postfix="4" reflect="1"/>
+    <xacro:ezgripper_knuckle prefix="${prefix}" postfix="1" reflectY="1" reflectZ="1" reflectR="1" mimic_test="false"/>
+    <xacro:ezgripper_knuckle prefix="${prefix}" postfix="2" reflectY="-1" reflectZ="1" reflectR="-1" mimic_test="true"/>
+    <xacro:ezgripper_knuckle prefix="${prefix}" postfix="3" reflectY="1" reflectZ="-1" reflectR="1" mimic_test="true"/>
+    <xacro:ezgripper_knuckle prefix="${prefix}" postfix="4" reflectY="-1" reflectZ="-1" reflectR="-1" mimic_test="true"/>
+    <xacro:ezgripper_knuckle_trans prefix="${prefix}" postfix="1"/>
+    <xacro:ezgripper_knuckle_trans prefix="${prefix}" postfix="2"/>
+    <xacro:ezgripper_knuckle_trans prefix="${prefix}" postfix="3"/>
+    <xacro:ezgripper_knuckle_trans prefix="${prefix}" postfix="4"/>
+    <xacro:gazebo_knuckle_jsp prefix="${prefix}" />
 </xacro:macro>
 <xacro:macro name="ezgripper_finger" params="prefix postfix reflect">

File: ezgripper_driver/urdf/ezgripper_quad_standalone.urdf.xacro (robot description, xacro)
@@ -6,7 +6,10 @@
 <xacro:include filename="$(find ezgripper_driver)/urdf/ezgripper_quad.urdf.xacro"/>
 <!-- Add the gripper -->
-<ezgripper_quad prefix="left" parent_link="base_link">
+<xacro:ezgripper_quad prefix="left" parent_link="base_link">
 <origin xyz="${ezgripper_offset_x} ${ezgripper_offset_y} ${ezgripper_offset_z}" rpy="0 0 0"/>
-</ezgripper_quad>
+</xacro:ezgripper_quad>
+<material name="red">
+  <color rgba="0.7 0.0 0.0 0.99"/>
+</material>
 <link name="world"/>
 <joint name="fixed" type="fixed">
